Commit message: feat: Massive update, sound part

File: ros/src/abot_description/urdf/abot.xacro (robot description, xacro)
@@ -12,7 +12,7 @@
 	<link name="abot_base">
 		<inertial>
-			<origin xyz="-0.020033 -0.0011051 0.056486" rpy="0 0 0"/>
-			<mass value="0.54627"/>
-			<inertia ixx="0.00061681" ixy="-1.7116E-06" ixz="-1.1044E-05" iyy="0.00061911" iyz="-8.1361E-09" izz="0.0011295"/>
+			<origin xyz="-0.017258 -0.00044491 0.079113" rpy="0 0 0"/>
+			<mass value="0.71798"/>
+			<inertia ixx="0.00077488" ixy="-3.248E-06" ixz="-9.2329E-06" iyy="0.00075836" iyz="2.2456E-06" izz="0.0014158"/>
 		</inertial>
 		<visual>

File: ros/src/abot_description/urdf/abot_sensors.xacro (robot description, xacro)
@@ -24,5 +24,5 @@
 	</link>
 	<joint name="lidar_to_base" type="fixed">
-		<origin xyz="-0.01 0 0.1419" rpy="0 0 ${PI}"/>
+		<origin xyz="-0.01 0 0.1849" rpy="0 0 ${PI}"/>
 		<parent link="abot_base"/>
 		<child link="abot_lidar"/>
